Commit message: Validate complete 6-DOF RoboCup arm
- import final 6-DOF arm joint chain and wrist geometry
- validate individual and simultaneous dual-arm motion
- validate 2.5 kg payload across all six arm DOFs
- validate loaded shoulder reach at 90 and 120 degrees
- validate 3.0 rad/s velocity ceiling across all 12 revolute joints
- validate 55/55/30/25/8/8 Nm effort ceilings
- preserve force-torque instrumentation and saturation models
- preserve shoulder-yaw external-wrench investigations
- preserve rejected and anomalous measurement attempts
- preserve raw velocity and torque logs
- preserve generated URDF/SDF validation models
- preserve all validation scripts
- add final motor-output envelope and electrical handoff dataset

File: ros2_ws/src/RoboticArm/urdf/robothath.urdf (robot description, URDF)
Before this commit: robot robothath, 20 links, 19 joints
Links:
- removed link l_wrist_roll_link
- removed link r_wrist_roll_link
- added link l_shoulder_link, mass 0.001
- added link r_shoulder_link, mass 0.001
- link l_forearm_link: mass 0.7675 -> 0.5888
- link l_wrist_link: mass 0.1 -> 0.1787; geometry collision mesh filename=package://robothath_description/meshes/l_wrist_link.stl; visual mesh filename=package://robothath_description/meshes/l_wrist_link.stl
- link r_forearm_link: mass 0.7675 -> 0.5888
- link r_wrist_link: mass 0.1 -> 0.1787; geometry collision mesh filename=package://robothath_description/meshes/r_wrist_link.stl; visual mesh filename=package://robothath_description/meshes/r_wrist_link.stl
Joints:
- removed joint l_gripper_mount_joint
- removed joint r_gripper_mount_joint
- added joint l_shoulder_roll_joint: type revolute, parent l_shoulder_link, child l_upper_arm_link, origin xyz=0.0000 0.0000 0.0000 rpy=0 0 0, axis 1 0 0, limit lower=-2.0944 upper=2.0944 effort=40 velocity=3.0
- added joint r_shoulder_roll_joint: type revolute, parent r_shoulder_link, child r_upper_arm_link, origin xyz=0.0000 0.0000 0.0000 rpy=0 0 0, axis 1 0 0, limit lower=-2.0944 upper=2.0944 effort=40 velocity=3.0
- joint l_base_mount_joint: origin xyz=0 0.0000 0 rpy=0 0 0 -> xyz=0.0000 0.0000 0.0000 rpy=0 0 0
- joint l_base_yaw_joint: origin xyz=0 0 0 rpy=0 0 0 -> xyz=0.0000 0.0000 0.0000 rpy=0 0 0
- joint l_elbow_pitch_joint: limit lower=-2.6180 upper=2.6180 effort=30 velocity=3.0 -> lower=-2.618 upper=2.618 effort=30 velocity=3.0; origin xyz=-0.342 0 0 rpy=0 0 0 -> xyz=-0.3420 0.0000 0.0000 rpy=0 0 0
- joint l_finger_inner_joint: origin xyz=0.003 0.0223 -0.130 rpy=0 0 0 -> xyz=0.0035 0.0189 -0.0710 rpy=0 0 0
- joint l_finger_outer_joint: origin xyz=0.003 -0.0175 -0.130 rpy=0 0 0 -> xyz=0.0035 -0.0209 -0.0710 rpy=0 0 0
- joint l_shoulder_pitch_joint: child l_upper_arm_link -> l_shoulder_link; origin xyz=0 0 -0.025 rpy=0 0 0 -> xyz=0.0000 0.0000 -0.0250 rpy=0 0 0
- joint l_wrist_joint: limit lower=-3.1416 upper=3.1416 effort=20 velocity=2.0 -> lower=-1.5708 upper=1.5708 effort=20 velocity=3.0; origin xyz=0 0 -0.275 rpy=0 0 0 -> xyz=-0.0003 0.0000 -0.2580 rpy=0 0 0
- joint l_wrist_roll_joint: axis 1 0 0 -> 0 0 1; child l_wrist_roll_link -> l_gripper_base; limit lower=-3.1416 upper=3.1416 effort=20 velocity=2.0 -> lower=-3.1416 upper=3.1416 effort=10 velocity=3.0; origin xyz=0 0 0 rpy=0 0 0 -> xyz=-0.0002 0.0034 -0.0760 rpy=0 0 0
- joint r_base_mount_joint: origin xyz=0 0.5236 0 rpy=0 0 0 -> xyz=0.0000 0.5236 0.0000 rpy=0 0 0
- joint r_base_yaw_joint: origin xyz=0 0 0 rpy=0 0 0 -> xyz=0.0000 0.0000 0.0000 rpy=0 0 0
- joint r_elbow_pitch_joint: limit lower=-2.6180 upper=2.6180 effort=30 velocity=3.0 -> lower=-2.618 upper=2.618 effort=30 velocity=3.0; origin xyz=-0.342 0 0 rpy=0 0 0 -> xyz=-0.3420 0.0000 0.0000 rpy=0 0 0
- joint r_finger_inner_joint: origin xyz=0.003 -0.0223 -0.130 rpy=0 0 0 -> xyz=0.0035 -0.0189 -0.0710 rpy=0 0 0
- joint r_finger_outer_joint: origin xyz=0.003 0.0175 -0.130 rpy=0 0 0 -> xyz=0.0035 0.0209 -0.0710 rpy=0 0 0
- joint r_shoulder_pitch_joint: child r_upper_arm_link -> r_shoulder_link; origin xyz=0 0 -0.025 rpy=0 0 0 -> xyz=0.0000 0.0000 -0.0250 rpy=0 0 0
- joint r_wrist_joint: limit lower=-3.1416 upper=3.1416 effort=20 velocity=2.0 -> lower=-1.5708 upper=1.5708 effort=20 velocity=3.0; origin xyz=0 0 -0.275 rpy=0 0 0 -> xyz=-0.0003 0.0000 -0.2580 rpy=0 0 0
- joint r_wrist_roll_joint: axis 1 0 0 -> 0 0 1; child r_wrist_roll_link -> r_gripper_base; limit lower=-3.1416 upper=3.1416 effort=20 velocity=2.0 -> lower=-3.1416 upper=3.1416 effort=10 velocity=3.0; origin xyz=0 0 0 rpy=0 0 0 -> xyz=-0.0002 -0.0034 -0.0760 rpy=0 0 0
